File: PCB/SnakeBoard.kicad_sch (KiCad schematic)
At the start: 192 parts, among them SW1 SW_Push, SW10 SW_Push, SW11 SW_Push, SW12 SW_Push, SW13 SW_Push, SW14 SW_Push, SW15 SW_Push, SW16 SW_Push, SW17 SW_Push, SW18 SW_Push, SW19 SW_Push, SW2 SW_Push, SW20 SW_Push, SW21 SW_Push, SW22 SW_Push, SW23 SW_Push, SW24 SW_Push, SW25 SW_Push, SW26 SW_Push, SW27 SW_Push, SW28 SW_Push, SW29 SW_Push, SW3 SW_Push, SW30 SW_Push, SW31 SW_Push, SW32 SW_Push, SW33 SW_Push, SW34 SW_Push, SW35 SW_Push, SW36 SW_Push, SW37 SW_Push, SW38 SW_Push, SW39 SW_Push, SW4 SW_Push, SW40 SW_Push, SW41 SW_Push, SW42 SW_Push, SW43 SW_Push, SW44 SW_Push, SW45 SW_Push, SW46 SW_Push, SW47 SW_Push, SW48 SW_Push, SW49 SW_Push, SW5 SW_Push, SW50 SW_Push, SW51 SW_Push, SW52 SW_Push, SW53 SW_Push, SW54 SW_Push, SW55 SW_Push, SW56 SW_Push, SW57 SW_Push, SW58 SW_Push, SW59 SW_Push, SW6 SW_Push, SW60 SW_Push, SW61 SW_Push, SW62 SW_Push, SW63 SW_Push, SW64 SW_Push, SW65 SW_Push, SW66 SW_Push, SW67 SW_Push, SW68 SW_Push, SW69 SW_Push, SW7 SW_Push, SW70 SW_Push, SW71 SW_Push, SW72 SW_Push, SW73 SW_Push, SW74 SW_Push, SW75 SW_Push, SW76 SW_Push, SW77 SW_Push, SW78 SW_Push, SW79 SW_Push, SW8 SW_Push, SW80 SW_Push, SW81 SW_Push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

Commit message: add teh schematic changes
Parts:
- added A2: RaspberryPi_Pico, Module:RaspberryPi_Pico_Common_Unspecified, symbol MCU_Module:RaspberryPi_Pico
- added U1: 74HC165, symbol 74xx:74HC165
Connections:
- net Row5: now reaches D11.1 (K), D17.1 (K), D23.1 (K), D29.1 (K), D35.1 (K), D41.1 (K), D47.1 (K), D5.1 (K), D53.1 (K), D59.1 (K), D65.1 (K), D75.1 (K), D77.1 (K), D83.1 (K), D89.1 (K), D95.1 (K)
- net Row4: now reaches D10.1 (K), D16.1 (K), D22.1 (K), D28.1 (K), D34.1 (K), D4.1 (K), D40.1 (K), D46.1 (K), D52.1 (K), D58.1 (K), D64.1 (K), D70.1 (K), D74.1 (K), D82.1 (K), D88.1 (K), D94.1 (K)
- net Row2: now reaches D14.1 (K), D2.1 (K), D20.1 (K), D26.1 (K), D32.1 (K), D38.1 (K), D44.1 (K), D50.1 (K), D56.1 (K), D62.1 (K), D68.1 (K), D72.1 (K), D8.1 (K), D80.1 (K), D86.1 (K), D92.1 (K)
- net Row3: now reaches D15.1 (K), D21.1 (K), D27.1 (K), D3.1 (K), D33.1 (K), D39.1 (K), D45.1 (K), D51.1 (K), D57.1 (K), D63.1 (K), D69.1 (K), D73.1 (K), D81.1 (K), D87.1 (K), D9.1 (K), D93.1 (K)
- net Row6: now reaches D12.1 (K), D18.1 (K), D24.1 (K), D30.1 (K), D36.1 (K), D42.1 (K), D48.1 (K), D54.1 (K), D6.1 (K), D60.1 (K), D66.1 (K), D76.1 (K), D78.1 (K), D84.1 (K), D90.1 (K), D96.1 (K)
- new net: A2.13 (GND), A2.18 (GND), A2.23 (GND), A2.28 (GND), A2.3 (GND), A2.38 (GND), A2.8 (GND)
- new net +5V: A2.40 (VBUS)
