File: PCB/SnakeBoard.kicad_sch (KiCad schematic)
At the start: 205 parts, among them J1 Conn_01x04_Pin, J2 Conn_01x04_Pin, SW1 SW_Push, SW10 SW_Push, SW11 SW_Push, SW12 SW_Push, SW13 SW_Push, SW14 SW_Push, SW15 SW_Push, SW16 SW_Push, SW17 SW_Push, SW18 SW_Push, SW19 SW_Push, SW2 SW_Push, SW20 SW_Push, SW21 SW_Push, SW22 SW_Push, SW23 SW_Push, SW24 SW_Push, SW25 SW_Push, SW26 SW_Push, SW27 SW_Push, SW28 SW_Push, SW29 SW_Push, SW3 SW_Push, SW30 SW_Push, SW31 SW_Push, SW32 SW_Push, SW33 SW_Push, SW34 SW_Push, SW35 SW_Push, SW36 SW_Push, SW37 SW_Push, SW38 SW_Push, SW39 SW_Push, SW4 SW_Push, SW40 SW_Push, SW41 SW_Push, SW42 SW_Push, SW43 SW_Push, SW44 SW_Push, SW45 SW_Push, SW46 SW_Push, SW47 SW_Push, SW48 SW_Push, SW49 SW_Push, SW5 SW_Push, SW50 SW_Push, SW51 SW_Push, SW52 SW_Push, SW53 SW_Push, SW54 SW_Push, SW55 SW_Push, SW56 SW_Push, SW57 SW_Push, SW58 SW_Push, SW59 SW_Push, SW6 SW_Push, SW60 SW_Push, SW61 SW_Push, SW62 SW_Push, SW63 SW_Push, SW64 SW_Push, SW65 SW_Push, SW66 SW_Push, SW67 SW_Push, SW68 SW_Push, SW69 SW_Push, SW7 SW_Push, SW70 SW_Push, SW71 SW_Push, SW72 SW_Push, SW73 SW_Push, SW74 SW_Push, SW75 SW_Push, SW76 SW_Push, SW77 SW_Push, SW78 SW_Push, SW79 SW_Push, SW8 SW_Push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

Commit message: Added the PCB remains the routing
Parts:
- removed D91, D92, D93, D94, D95, D96: D, symbol Device:D
- removed SW91, SW92, SW93, SW94, SW95, SW96: SW_Push, symbol Switch:SW_Push
- A2: footprint Module:RaspberryPi_Pico_Common_Unspecified -> test:RaspberryPi_Pico_Common_Unspecified
- D1, D10, D11, D12, D13, D14, D15, D16, D17, D18, D19, D2, D20, D21, D22, D23, D24, D25, D26, D27, D28, D29, D3, D30, D31, D32, D33, D34, D35, D36, D37, D38, D39, D4, D40, D41, D42, D43, D44, D45, D46, D47, D48, D49, D5, D50, D51, D52, D53, D54, D55, D56, D57, D58, D59, D6, D60, D61, D62, D63, D64, D65, D66, D67, D68, D69, D7, D70, D71, D72, D73, D74, D75, D76, D77, D78, D79, D8, D80, D81, D82, D83, D84, D85, D86, D87, D88, D89, D9, D90: footprint (none) -> Diode_THT:D_DO-35_SOD27_P7.62mm_Horizontal
- J1, J2: footprint (none) -> test:SSD1306_0.96_Oled
- SW1, SW10, SW11, SW12, SW13, SW14, SW15, SW16, SW17, SW18, SW19, SW2, SW20, SW21, SW22, SW23, SW24, SW25, SW26, SW27, SW28, SW29, SW3, SW30, SW31, SW32, SW33, SW34, SW35, SW36, SW37, SW38, SW39, SW4, SW40, SW41, SW42, SW43, SW44, SW45, SW46, SW47, SW48, SW49, SW5, SW50, SW51, SW52, SW53, SW54, SW55, SW56, SW57, SW58, SW59, SW6, SW60, SW61, SW62, SW63, SW64, SW65, SW66, SW67, SW68, SW69, SW7, SW70, SW71, SW72, SW73, SW74, SW75, SW76, SW77, SW78, SW79, SW8, SW80, SW81, SW82, SW83, SW84, SW85, SW86, SW87, SW88, SW89, SW9, SW90: footprint (none) -> test:SW_Cherry_MX_1.00u_PCB
- SW97: footprint (none) -> test:RotaryEncoder_Alps_EC12E-Switch_Vertical_H20mm
- U1: footprint (none) -> Package_DIP:DIP-16_W7.62mm
Connections:
- net Col1: now also SW15.1, SW30.1, SW45.1, SW60.1, SW75.1, SW90.1
- net Col10: now also SW21.1, SW36.1, SW51.1, SW6.1, SW66.1, SW81.1; no longer SW22.1, SW37.1, SW52.1, SW67.1, SW7.1, SW82.1
- net Col11: now also SW20.1, SW35.1, SW5.1, SW50.1, SW65.1, SW80.1; no longer SW21.1, SW36.1, SW51.1, SW6.1, SW66.1, SW81.1
- net Col12: now also SW19.1, SW34.1, SW4.1, SW49.1, SW64.1, SW79.1; no longer SW20.1, SW35.1, SW5.1, SW50.1, SW65.1, SW80.1
- net Col13: now also SW18.1, SW3.1, SW33.1, SW48.1, SW63.1, SW78.1; no longer SW19.1, SW34.1, SW4.1, SW49.1, SW64.1, SW79.1
- net Col14: now also SW17.1, SW2.1, SW32.1, SW47.1, SW62.1, SW77.1; no longer SW18.1, SW3.1, SW33.1, SW48.1, SW63.1, SW78.1
- net Col15: now also SW1.1, SW16.1, SW31.1, SW46.1, SW61.1, SW76.1; no longer SW17.1, SW2.1, SW32.1, SW47.1, SW62.1, SW77.1
- net Col16: no longer SW1.1, SW16.1, SW31.1, SW46.1, SW61.1, SW76.1
- net Col2: now also SW14.1, SW29.1, SW44.1, SW59.1, SW74.1, SW89.1; no longer SW15.1, SW30.1, SW45.1, SW60.1, SW75.1, SW90.1
- net Col3: now also SW13.1, SW28.1, SW43.1, SW58.1, SW73.1, SW88.1; no longer SW14.1, SW29.1, SW44.1, SW59.1, SW74.1, SW89.1
- net Col4: now also SW12.1, SW27.1, SW42.1, SW57.1, SW72.1, SW87.1; no longer SW13.1, SW28.1, SW43.1, SW58.1, SW73.1, SW88.1
- net Col5: now also SW11.1, SW26.1, SW41.1, SW56.1, SW71.1, SW86.1; no longer SW12.1, SW27.1, SW42.1, SW57.1, SW72.1, SW87.1
- net Col6: now also SW10.1, SW25.1, SW40.1, SW55.1, SW70.1, SW85.1; no longer SW11.1, SW26.1, SW41.1, SW56.1, SW71.1, SW86.1
- net Col7: now also SW24.1, SW39.1, SW54.1, SW69.1, SW84.1, SW9.1; no longer SW10.1, SW25.1, SW40.1, SW55.1, SW70.1, SW85.1
- net Col8: now also SW23.1, SW38.1, SW53.1, SW68.1, SW8.1, SW83.1; no longer SW24.1, SW39.1, SW54.1, SW69.1, SW84.1, SW9.1
- net Col9: now also SW22.1, SW37.1, SW52.1, SW67.1, SW7.1, SW82.1; no longer SW23.1, SW38.1, SW53.1, SW68.1, SW8.1, SW83.1
