File: PCB/SnakeBoard.kicad_pcb (KiCad board)
At the start: 2 copper layers, 315 x 152.4 mm, 193 parts, among them J1 Conn_01x04_Pin, J2 Conn_01x04_Pin, SW1 SW_Push, SW10 SW_Push, SW11 SW_Push, SW12 SW_Push, SW13 SW_Push, SW14 SW_Push, SW15 SW_Push, SW16 SW_Push, SW17 SW_Push, SW18 SW_Push, SW19 SW_Push, SW2 SW_Push, SW20 SW_Push, SW21 SW_Push, SW22 SW_Push, SW23 SW_Push, SW24 SW_Push, SW25 SW_Push, SW26 SW_Push, SW27 SW_Push, SW28 SW_Push, SW29 SW_Push, SW3 SW_Push, SW30 SW_Push, SW31 SW_Push, SW32 SW_Push, SW33 SW_Push, SW34 SW_Push, SW35 SW_Push, SW36 SW_Push, SW37 SW_Push, SW38 SW_Push, SW39 SW_Push, SW4 SW_Push, SW40 SW_Push, SW41 SW_Push, SW42 SW_Push, SW43 SW_Push, SW44 SW_Push, SW45 SW_Push, SW46 SW_Push, SW47 SW_Push, SW48 SW_Push, SW49 SW_Push, SW5 SW_Push, SW50 SW_Push, SW51 SW_Push, SW52 SW_Push, SW53 SW_Push, SW54 SW_Push, SW55 SW_Push, SW56 SW_Push, SW57 SW_Push, SW58 SW_Push, SW59 SW_Push, SW6 SW_Push, SW60 SW_Push, SW61 SW_Push, SW62 SW_Push, SW63 SW_Push, SW64 SW_Push, SW65 SW_Push, SW66 SW_Push, SW67 SW_Push, SW68 SW_Push, SW69 SW_Push, SW7 SW_Push, SW70 SW_Push, SW71 SW_Push, SW72 SW_Push, SW73 SW_Push, SW74 SW_Push, SW75 SW_Push, SW76 SW_Push, SW77 SW_Push, SW78 SW_Push, SW79 SW_Push, SW8 SW_Push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

Commit message: Finished the PCB and it is all done.
Parts:
- A2: moved to F.Cu
- moved D2 286.4 mm to (31.7, 70.5)
- moved D8 286.4 mm to (317.4, 51.5)
- moved SW16 286.4 mm to (38.1, 57.1)
- moved SW17 286.4 mm to (323.9, 38.1)
- moved D3 281.6 mm to (36.5, 89.6)
- moved D9 281.6 mm to (317.4, 70.5)
- moved SW31 281.6 mm to (42.9, 76.2)
- moved SW32 281.6 mm to (323.9, 57.1)
- moved SW46 279.3 mm to (45.2, 95.2)
- moved SW47 279.3 mm to (323.9, 76.2)
- moved D10 279.3 mm to (317.4, 89.6)
- moved D4 279.3 mm to (38.8, 108.7)
- turned A2 to 90 degrees
Routing:
- net Row6: track 0.00 -> 861.4 mm, vias 0 -> 3
- net +5V: track 0.00 -> 592.5 mm, vias 0 -> 25
- net Col1: track 0.00 -> 491.3 mm, vias 0 -> 3
- net Row5: track 0.00 -> 484.0 mm, vias 0 -> 2
- net Row4: track 0.00 -> 462.0 mm, vias 0 -> 6
- net Col14: track 0.00 -> 421.9 mm, vias 0 -> 1
- net Row3: track 0.00 -> 412.4 mm, vias 0 -> 5
- net Col7: track 0.00 -> 396.4 mm, vias 0 -> 1
- net Row1: track 0.00 -> 389.3 mm, vias 0 -> 4
- net Row2: track 0.00 -> 388.6 mm, vias 0 -> 6
- net Col3: track 0.00 -> 384.0 mm
- net Col2: track 0.00 -> 365.5 mm
- net Col8: track 0.00 -> 355.1 mm, vias 0 -> 3
- net Col4: track 0.00 -> 351.3 mm
- net Col9: track 0.00 -> 339.2 mm, vias 0 -> 3
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- added copper zone on B.Cu, net GND
